File: Hardware/wireless_BLE.kicad_sch (KiCad schematic)
At the start: 5 parts

Commit message: wired USB battery charger
Connections:
- net ANT renamed nrf_ANT
Changed lines of the file:
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@@
 		)
 	)
-	(global_label "ANT"
+	(global_label "nrf_ANT"
 		(shape input)
 		(at 96.52 101.6 180)
@@
 		)
 		(property "Intersheetrefs" "${INTERSHEET_REFS}"
-			(at 90.1481 101.6 0)
+			(at 86.5196 101.6 0)
 			(effects
 				(font

Commit message: finish draft of power schematic
Parts:
- gave numbers to parts that had none: 1
Changed lines of the file:
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@@
 		(on_board yes)
 		(dnp no)
-		(property "Reference" "IFA?"
+		(property "Reference" "IFA1"
 			(at 175.006 87.376 90)
 			(effects
@@
 			(project "hornet_kb"
 				(path "/c35084ab-104c-4a4c-9388-a839989b8e3d/8c7a30bd-1c2f-4bc6-8f52-c45519217f8c"
-					(reference "IFA?")
+					(reference "IFA1")
 					(unit 1)
 				)

Commit message: Complete first ROUGH draft of schematic
Parts:
- removed IFA1: ~, symbol Device:IFA
Changed lines of the file:
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@@
 	(wire
 		(pts
-			(xy 171.45 109.22) (xy 171.45 104.14)
+			(xy 107.95 101.6) (xy 96.52 101.6)
 		)
 		(stroke
@@
 		)
 	)
-	(wire
-		(pts
-			(xy 107.95 101.6) (xy 96.52 101.6)
-		)
-		(stroke
-			(width 0)
-			(type default)
-		)
-	)
 	(global_label "nrf_ANT"
 		(shape input)
@@
 				(path "/c35084ab-104c-4a4c-9388-a839989b8e3d/8c7a30bd-1c2f-4bc6-8f52-c45519217f8c"
 					(reference "#PWR013")
-					(unit 1)
-				)
-			)
-		)
-	)
-	(symbol
-		(lib_id "power:GND")
-		(at 171.45 109.22 0)
-		(unit 1)
-		(exclude_from_sim no)
-		(in_bom yes)
-		(on_board yes)
-		(dnp no)
-		(fields_autoplaced yes)
-		(property "Reference" "#PWR018"
-			(at 171.45 115.57 0)
-			(effects
-				(font
-					(size 1.27 1.27)
-				)
-				(hide yes)
-			)
-		)
-		(property "Value" "GND"
-			(at 171.45 114.3 0)
-			(effects
-				(font
-					(size 1.27 1.27)
-				)
-			)
-		)
-		(property "Footprint" ""
-			(at 171.45 109.22 0)
-			(effects
-				(font
-					(size 1.27 1.27)
-				)
-				(hide yes)
-			)
-		)
-		(property "Datasheet" ""
-			(at 171.45 109.22 0)
-			(effects
-				(font
-					(size 1.27 1.27)
-				)
-				(hide yes)
-			)
-		)
-		(property "Description" "Power symbol creates a global label with name \"GND\" , ground"
-			(at 171.45 109.22 0)
-			(effects
-				(font
-					(size 1.27 1.27)
-				)
-				(hide yes)
-			)
-		)
-		(pin "1"
-		)
-		(instances
-			(project "hornet_kb"
-				(path "/c35084ab-104c-4a4c-9388-a839989b8e3d/8c7a30bd-1c2f-4bc6-8f52-c45519217f8c"
-					(reference "#PWR018")
 					(unit 1)
 				)
@@
 					(unit 1)
 				)
-			)
-		)
-	)
-	(symbol
-		(lib_name "IFA_1")
-		(lib_id "Device:IFA")
-		(at 177.8 96.52 270)
-		(mirror x)
-		(unit 1)
-		(exclude_from_sim no)
-		(in_bom yes)
-		(on_board yes)
-		(dnp no)
-		(property "Reference" "IFA1"
-			(at 175.006 87.376 90)
-			(effects
-				(font
-					(size 1.27 1.27)
-				)
-			)
-		)
-		(property "Value" "~"
-			(at 175.26 86.36 90)
-			(effects
-				(font
-					(size 1.27 1.27)
-				)
-				(hide yes)
-			)
-		)
-		(property "Footprint" ""
-			(at 177.8 96.52 0)
-			(effects
-				(font
-					(size 1.27 1.27)
-				)
-				(hide yes)
-			)
-		)
-		(property "Datasheet" ""
-			(at 177.8 96.52 0)
-			(effects
-				(font
-					(size 1.27 1.27)
-				)
-				(hide yes)
-			)
-		)
-		(property "Description" ""
-			(at 177.8 96.52 0)
-			(effects
-				(font
-					(size 1.27 1.27)
-				)
-				(hide yes)
-			)
-		)
-		(pin ""
-		)
-		(pin ""
-		)
-		(instances
-			(project "hornet_kb"
-				(path "/c35084ab-104c-4a4c-9388-a839989b8e3d/8c7a30bd-1c2f-4bc6-8f52-c45519217f8c"
-					(reference "IFA1")
-					(unit 1)
-				)
