File: Hardware/power_management.kicad_sch (KiCad schematic)
At the start: 37 parts, among them J2 Conn_01x03, SW27 SW_DPDT_x2, U2 BQ24040, U3 BQ51050BRHL, U4 AP22814BW5, U5 TPS2116DRL

Commit message: Added jumper to override power switch
Parts:
- added JP4: PWR_SWITCH, Jumper:SolderJumper-2_P1.3mm_Open_TrianglePad1.0x1.5mm, symbol Jumper:SolderJumper_2_Open
- SW27: footprint Button_Switch_THT:SW_CK_JS202011CQN_DPDT_Straight -> ScottoKeebs_Miscellaneous:SW_CK_JS202011CQN_DPDT_Straight
Connections:
- net +BATT: now also JP4.1 (A)
- net at JP1.1 (A), SW27.3 (C), SW27.6 (C): now also JP4.2 (B)
Changed lines of the file:
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@@
 	)
 	(junction
+		(at 220.98 110.49)
+		(diameter 0)
+		(color 0 0 0 0)
+	)
+	(junction
 		(at 196.85 115.57)
 		(diameter 0)
@@
 	)
 	(junction
+		(at 245.11 110.49)
+		(diameter 0)
+		(color 0 0 0 0)
+	)
+	(junction
 		(at 256.54 110.49)
 		(diameter 0)
@@
 	(wire
 		(pts
-			(xy 198.12 110.49) (xy 226.06 110.49)
+			(xy 198.12 110.49) (xy 220.98 110.49)
 		)
 		(stroke
@@
 	(wire
 		(pts
+			(xy 237.49 128.27) (xy 245.11 128.27)
+		)
+		(stroke
+			(width 0)
+			(type default)
+		)
+	)
+	(wire
+		(pts
 			(xy 80.01 130.81) (xy 74.93 130.81)
 		)
@@
 	(wire
 		(pts
-			(xy 238.76 110.49) (xy 246.38 110.49)
+			(xy 238.76 110.49) (xy 245.11 110.49)
 		)
 		(stroke
@@
 	(wire
 		(pts
+			(xy 229.87 128.27) (xy 220.98 128.27)
+		)
+		(stroke
+			(width 0)
+			(type default)
+		)
+	)
+	(wire
+		(pts
 			(xy 238.76 116.84) (xy 238.76 119.38)
 		)
@@
 	(wire
 		(pts
+			(xy 245.11 110.49) (xy 246.38 110.49)
+		)
+		(stroke
+			(width 0)
+			(type default)
+		)
+	)
+	(wire
+		(pts
 			(xy 90.17 142.24) (xy 90.17 146.05)
 		)
@@
 	(wire
 		(pts
+			(xy 220.98 128.27) (xy 220.98 110.49)
+		)
+		(stroke
+			(width 0)
+			(type default)
+		)
+	)
+	(wire
+		(pts
 			(xy 119.38 130.81) (xy 121.92 130.81)
 		)
@@
 	(wire
 		(pts
+			(xy 220.98 110.49) (xy 226.06 110.49)
+		)
+		(stroke
+			(width 0)
+			(type default)
+		)
+	)
+	(wire
+		(pts
 			(xy 189.23 143.51) (xy 189.23 148.59)
 		)
@@
 	(wire
 		(pts
+			(xy 245.11 128.27) (xy 245.11 110.49)
+		)
+		(stroke
+			(width 0)
+			(type default)
+		)
+	)
+	(wire
+		(pts
 			(xy 240.03 149.86) (xy 240.03 151.13)
 		)
@@
 	)
 	(symbol
+		(lib_id "Jumper:SolderJumper_2_Open")
+		(at 233.68 128.27 0)
+		(unit 1)
+		(exclude_from_sim no)
+		(in_bom no)
+		(on_board yes)
+		(dnp no)
+		(property "Reference" "JP4"
+			(at 228.854 129.794 0)
+			(effects
+				(font
+					(size 1.27 1.27)
+				)
+				(justify left)
+			)
+		)
+		(property "Value" "PWR_SWITCH"
+			(at 235.458 130.048 0)
+			(effects
+				(font
+					(size 1.27 1.27)
+				)
+				(justify left)
+			)
+		)
+		(property "Footprint" "Jumper:SolderJumper-2_P1.3mm_Open_TrianglePad1.0x1.5mm"
+			(at 233.68 128.27 0)
+			(effects
+				(font
+					(size 1.27 1.27)
+				)
+				(hide yes)
+			)
+		)
+		(property "Datasheet" "~"
+			(at 233.68 128.27 0)
+			(effects
+				(font
+					(size 1.27 1.27)
+				)
+				(hide yes)
+			)
+		)
+		(property "Description" "Solder Jumper, 2-pole, open"
+			(at 233.68 128.27 0)
+			(effects
+				(font
+					(size 1.27 1.27)
+				)
+				(hide yes)
+			)
+		)
+		(pin "1"
+		)
+		(pin "2"
+		)
+		(instances
+			(project "hornet_kb"
+				(path "/c35084ab-104c-4a4c-9388-a839989b8e3d/20e65fb9-037d-41f9-856c-d800ba40b4b1"
+					(reference "JP4")
+					(unit 1)
+				)
+			)
+		)
+	)
+	(symbol
 		(lib_id "power:GND")
 		(at 222.25 156.21 0)
@@
 			)
 		)
-		(property "Footprint" "Button_Switch_THT:SW_CK_JS202011CQN_DPDT_Straight"
+		(property "Footprint" "ScottoKeebs_Miscellaneous:SW_CK_JS202011CQN_DPDT_Straight"
 			(at 233.68 114.3 0)
 			(effects
@@
 			)
 		)
-		(property "Footprint" "Button_Switch_THT:SW_CK_JS202011CQN_DPDT_Straight"
+		(property "Footprint" "ScottoKeebs_Miscellaneous:SW_CK_JS202011CQN_DPDT_Straight"
 			(at 233.68 105.41 0)
 			(effects
